Commit message: Tristan worked to fix transforms and launch settings

File: robot_2024_description/urdf/camera_1.urdf (robot description, URDF)
Before this commit: robot cubert_1, 2 links, 1 joints
Links:
- added link camera_1_plane
- link base_link_1: geometry collision mesh filename=package://robot_2024_description/meshes/base_link.stl; visual mesh filename=package://robot_2024_description/meshes/base_link.stl
Joints:
- added joint camera2camera: type fixed, parent camera_1, child camera_1_plane, origin xyz=0 0 0 rpy=0 0 3.14
- joint b2c1: origin xyz=0.1 -0.25 0.1 rpy=0 0 1.57 -> xyz=0.07008632370852994 -0.12291145073927642 -0.3242521119533219 rpy=-0.007984225556421502 1.080362624275041 1.570788528447058; parent camera_1 -> camera_1_plane

File: robot_2024_description/urdf/camera_2.urdf (robot description, URDF)
Before this commit: robot cubert_2, 2 links, 1 joints
Links:
- added link camera_2_plane
- link base_link_2: geometry collision mesh filename=package://robot_2024_description/meshes/base_link.stl; visual mesh filename=package://robot_2024_description/meshes/base_link.stl
Joints:
- added joint camera2camera: type fixed, parent camera_2, child camera_2_plane, origin xyz=0 0 0 rpy=0 0 3.14
- joint b2c2: origin xyz=0.1 -0.25 0.1 rpy=0 0 1.57 -> xyz=-0.079 -0.068 -0.326 rpy=0.000 1.066 0.000

File: robot_2024_description/urdf/robot_2024.urdf (robot description, URDF)
Before this commit: robot robot_2024, 2 links, 1 joints
Links:
- added link c1
- added link c2
Joints:
- added joint b2c1_test: type fixed, parent base_link, child c1, origin xyz=-0.22814 0.068 0.2617 rpy=-2.06123 -3.14957 1.5708
- added joint b2c2_test: type fixed, parent base_link, child c2, origin xyz=-0.247 0.068 0.2261 rpy=0.0 -1.0664 0.0
