Commit message: Updates from code review

File: src/robot_2024_description/urdf/robot_2024.urdf (robot description, URDF)
Before this commit: robot robot_2024, 4 links, 3 joints
Links:
- added link rs_cam_1_link
Joints:
- added joint b2realsense: type fixed, parent base_link, child rs_cam_1_link, origin xyz=0.32 0.068 0.17 rpy=0.0 0.122173 0.0
