Commit message: Update camera configurations and deployment scripts; adjust file permissions and add Docker support

File: src/robot_2025_description/urdf/camera_1.urdf (robot description, URDF)
Before this commit: robot camera_1, 3 links, 2 joints
Joints:
- joint b2c1: origin xyz=0.07008632370852994 -0.12291145073927642 -0.3242521119533219 rpy=-0.007984225556421502 1.080362624275041 1.570788528447058 -> xyz=0.191 -0.283 -0.299 rpy=0.0 -1.57 0.0

File: src/robot_2025_description/urdf/camera_2.urdf (robot description, URDF)
Before this commit: robot camera_2, 3 links, 2 joints
Joints:
- joint b2c2: origin xyz=-0.079 -0.068 -0.326 rpy=0.000 1.066 0.000 -> xyz=0.191 0.283 -0.299 rpy=0.0 -1.57 0.0
