Commit message: Updates from testing

File: src/robot_2025_description/urdf/robot_2025.urdf (robot description, URDF)
Before this commit: robot robot_2025, 5 links, 4 joints
Links:
- removed link arm_link
- added link elevator_link; collision mesh filename=package://robot_2025_description/meshes/wrist.stl; visual mesh filename=package://robot_2025_description/meshes/wrist.stl
Joints:
- removed joint arm_joint
- added joint elevator_joint: type prismatic, parent base_link, child elevator_link, origin xyz=-0.146 0 0.261 rpy=0 0 0, axis 0 1 0, limit lower=-2.0 upper=0.07 effort=100.0 velocity=1.0
